File: AddOns/RelayBoard/RelayBoard.sch (KiCad schematic (older format))
At the start: 36 parts, among them P1 CONN_01X04, P2 CONN_01X06, P3 CONN_01X02, P4 CONN_01X08, Q1 BC817, Q2 BC817, Q3 BC817, Q4 BC817, SW1 SPST, SW2 SPST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

Commit message: fix layout problems
Parts:
- removed U1: MCP1703CB, SMD:SOT-23-3, symbol MCP1754ST-1802E/MB
- added U1: MCP1703-SOT23-3, SMD:SOT-23-3, symbol MCP1703-SOT23-3
- Q1, Q2, Q3, Q4: symbol Q_NPN_BCE -> Q_NPN_BEC
Connections:
- net +3V3: now also U1.2 (Vout)
- net +5V: now also U1.3 (Vin)
- net GND: now also Q1.2 (E), Q2.2 (E), Q3.2 (E), Q4.2 (E), U1.1 (GND); no longer Q1.3 (E), Q2.3 (E), Q3.3 (E), Q4.3 (E)
- net at D1.2 (A), D2.1 (K), P4.2 (P2): now also Q1.3 (C); no longer Q1.2 (C)
- net at D3.2 (A), D4.1 (K), P4.4 (P4): now also Q2.3 (C); no longer Q2.2 (C)
- net at D5.2 (A), D6.1 (K), P4.6 (P6): now also Q3.3 (C); no longer Q3.2 (C)
- net at D7.2 (A), D8.1 (K), P4.8 (P8): now also Q4.3 (C); no longer Q4.2 (C)
Other:
- moved on the sheet: C1
Changed lines of the file:
@@
 LIBS:contrib
 LIBS:valves
+LIBS:cc1101
 LIBS:RelayBoard-cache
 EELAYER 25 0
@@
 Title "Relay Board"
 Date ""
-Rev "V1.0"
+Rev "V1.1"
 Comp ""
 Comment1 ""
@@
 L C_Small C1
 U 1 1 5988E3C6
-P 3250 1800
-F 0 "C1" H 3260 1870 50  0000 L CNN
-F 1 "1µF" H 3260 1720 50  0000 L CNN
-F 2 "Capacitors_SMD:C_0805" H 3250 1800 50  0001 C CNN
-F 3 "" H 3250 1800 50  0000 C CNN
-	1    3250 1800
+P 3050 1800
+F 0 "C1" H 3060 1870 50  0000 L CNN
+F 1 "1µF" H 3060 1720 50  0000 L CNN
+F 2 "Capacitors_SMD:C_0805" H 3050 1800 50  0001 C CNN
+F 3 "" H 3050 1800 50  0000 C CNN
+	1    3050 1800
 	1    0    0    -1
 $EndComp
@@
 $EndComp
 $Comp
-L MCP1754ST-1802E/MB U1
-U 1 1 5988E760
-P 3700 1600
-F 0 "U1" H 3800 1450 50  0000 C CNN
-F 1 "MCP1703CB" H 3700 1750 50  0000 C CNN
-F 2 "SMD:SOT-23-3" H 3700 1600 50  0001 C CNN
-F 3 "" H 3700 1600 50  0000 C CNN
-	1    3700 1600
-	1    0    0    -1
-$EndComp
-$Comp
 L GND #PWR03
 U 1 1 5988EA70
-P 3250 1950
-F 0 "#PWR03" H 3250 1700 50  0001 C CNN
-F 1 "GND" H 3250 1800 50  0000 C CNN
-F 2 "" H 3250 1950 50  0000 C CNN
-F 3 "" H 3250 1950 50  0000 C CNN
-	1    3250 1950
+P 3050 1950
+F 0 "#PWR03" H 3050 1700 50  0001 C CNN
+F 1 "GND" H 3050 1800 50  0000 C CNN
+F 2 "" H 3050 1950 50  0000 C CNN
+F 3 "" H 3050 1950 50  0000 C CNN
+	1    3050 1950
 	1    0    0    -1
 $EndComp
@@
 L GND #PWR04
 U 1 1 5988EA9C
-P 3700 1950
-F 0 "#PWR04" H 3700 1700 50  0001 C CNN
-F 1 "GND" H 3700 1800 50  0000 C CNN
-F 2 "" H 3700 1950 50  0000 C CNN
-F 3 "" H 3700 1950 50  0000 C CNN
-	1    3700 1950
+P 3600 1950
+F 0 "#PWR04" H 3600 1700 50  0001 C CNN
+F 1 "GND" H 3600 1800 50  0000 C CNN
+F 2 "" H 3600 1950 50  0000 C CNN
+F 3 "" H 3600 1950 50  0000 C CNN
+	1    3600 1950
 	1    0    0    -1
 $EndComp
@@
 $EndComp
 Wire Wire Line
-	3250 1900 3250 1950
-Wire Wire Line
-	3700 1800 3700 1950
-Wire Wire Line
 	4100 1900 4100 1950
 Wire Wire Line
 	4400 1900 4400 1950
-Wire Wire Line
-	3400 1600 2650 1600
 Wire Wire Line
 	4400 1500 4400 1700
 Connection ~ 4400 1600
-Wire Wire Line
-	4100 1700 4100 1600
-Connection ~ 4100 1600
-Wire Wire Line
-	3250 1500 3250 1700
-Connection ~ 3250 1600
 $Comp
 L +3.3V #PWR07
@@
 	1    0    0    -1
 $EndComp
-Wire Wire Line
-	4000 1600 4400 1600
 $Comp
 L +3.3V #PWR08
@@
 	2750 2650 2750 2600
 $Comp
-L Q_NPN_BCE Q1
+L Q_NPN_BEC Q1
 U 1 1 5988F318
 P 6000 1900
@@
 L +5V #PWR09
 U 1 1 59890598
-P 3250 1500
-F 0 "#PWR09" H 3250 1350 50  0001 C CNN
-F 1 "+5V" H 3250 1640 50  0000 C CNN
-F 2 "" H 3250 1500 50  0000 C CNN
-F 3 "" H 3250 1500 50  0000 C CNN
-	1    3250 1500
+P 3050 1500
+F 0 "#PWR09" H 3050 1350 50  0001 C CNN
+F 1 "+5V" H 3050 1640 50  0000 C CNN
+F 2 "" H 3050 1500 50  0000 C CNN
+F 3 "" H 3050 1500 50  0000 C CNN
+	1    3050 1500
 	1    0    0    -1
 $EndComp
@@
 $EndComp
 $Comp
-L Q_NPN_BCE Q2
+L Q_NPN_BEC Q2
 U 1 1 59899956
 P 7300 3000
@@
 $EndComp
 $Comp
-L Q_NPN_BCE Q3
+L Q_NPN_BEC Q3
 U 1 1 5989C843
 P 6000 4150
@@
 $EndComp
 $Comp
-L Q_NPN_BCE Q4
+L Q_NPN_BEC Q4
 U 1 1 598A027C
 P 7300 5200
@@
 Wire Wire Line
 	8300 3400 8600 3400
+$Comp
+L MCP1703-SOT23-3 U1
+U 1 1 5996F7A2
+P 3600 1400
+F 0 "U1" H 3750 950 60  0000 C CNN
+F 1 "MCP1703-SOT23-3" H 3600 1400 60  0000 C CNN
+F 2 "SMD:SOT-23-3" H 3600 1400 60  0001 C CNN
+F 3 "" H 3600 1400 60  0000 C CNN
+	1    3600 1400
+	1    0    0    -1
+$EndComp
+Wire Wire Line
+	4050 1600 4400 1600
+Wire Wire Line
+	4100 1700 4100 1600
+Connection ~ 4100 1600
+Wire Wire Line
+	2650 1600 3150 1600
+Wire Wire Line
+	3050 1500 3050 1700
+Connection ~ 3050 1600
+Wire Wire Line
+	3050 1950 3050 1900
 $EndSCHEMATC
