File: AddOns/RelayBoard/RelayBoard.kicad_pcb (KiCad board)
At the start: 2 copper layers, 20 x 30 mm, 38 parts, among them P1 CONN_01X04, P2 CONN_01X06, P3 CONN_01X02, P4 CONN_01X08, Q1 BC817, Q2 BC817, Q3 BC817, Q4 BC817, SW1 SPST, SW2 SPST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

Commit message: fix layout problems
Parts:
- U1: value MCP1703CB -> MCP1703-SOT23-3
- turned U1 to 270 degrees
Connections:
- Q1 pad 2: Net-(D1-Pad2) -> GND
- Q1 pad 3: GND -> Net-(D1-Pad2)
- Q2 pad 2: Net-(D3-Pad2) -> GND
- Q2 pad 3: GND -> Net-(D3-Pad2)
- Q3 pad 2: Net-(D5-Pad2) -> GND
- Q3 pad 3: GND -> Net-(D5-Pad2)
- Q4 pad 2: Net-(D7-Pad2) -> GND
- Q4 pad 3: GND -> Net-(D7-Pad2)
- U1 pad 1: +5V -> GND
- U1 pad 2: GND -> +3V3
- U1 pad 3: +3V3 -> +5V
Routing:
- net Net-(D5-Pad2): track 13.0 -> 18.0 mm, vias 1 -> 2
- net Net-(D7-Pad2): track 12.8 -> 17.6 mm, vias 1 -> 2
- net Net-(D1-Pad2): track 13.4 -> 17.8 mm, vias 1 -> 2
- net Net-(D3-Pad2): track 13.4 -> 17.3 mm, vias 1 -> 2
- net GND: track 17.9 -> 14.7 mm
- net +5V: track 64.4 -> 63.4 mm
- net Net-(P1-Pad3): track 13.1 -> 12.1 mm
Other:
- board text added: "HMSensor Relay Board V1.1"
- board text removed: "HMSensor Relay Board V1.0"

Commit message: I²C V1.1 Relay V1.1
Changed lines of the file:
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@@
     (links 66)
     (no_connects 0)
-    (area 162.325857 91.995866 193.766834 128.991)
+    (area 169.924999 94.924999 190.075001 125.075001)
     (thickness 1.6)
     (drawings 25)
@@
     (effects (font (size 0.6 0.6) (thickness 0.1)))
   )
-  (gr_text T4 (at 175.9585 122.428) (layer F.SilkS)
+  (gr_text T1 (at 175.9585 122.428) (layer F.SilkS)
     (effects (font (size 0.6 0.6) (thickness 0.1)))
   )
-  (gr_text T3 (at 178.4985 122.4915) (layer F.SilkS)
+  (gr_text T2 (at 178.4985 122.4915) (layer F.SilkS)
     (effects (font (size 0.6 0.6) (thickness 0.1)))
   )
-  (gr_text T2 (at 181.0385 122.428) (layer F.SilkS)
+  (gr_text T3 (at 181.0385 122.428) (layer F.SilkS)
     (effects (font (size 0.6 0.6) (thickness 0.1)))
   )
-  (gr_text T1 (at 183.5785 122.428) (layer F.SilkS)
+  (gr_text T4 (at 183.5785 122.428) (layer F.SilkS)
     (effects (font (size 0.6 0.6) (thickness 0.1)))
   )
-  (gr_text R4 (at 186.055 122.428) (layer F.SilkS)
+  (gr_text R1 (at 186.055 122.428) (layer F.SilkS)
     (effects (font (size 0.6 0.6) (thickness 0.1)))
   )
-  (gr_text R3 (at 187.7695 122.7455 45) (layer F.SilkS)
+  (gr_text R2 (at 187.7695 122.7455 45) (layer F.SilkS)
     (effects (font (size 0.6 0.6) (thickness 0.1)))
   )
-  (gr_text R2 (at 187.2615 121.158 90) (layer F.SilkS)
+  (gr_text R3 (at 187.2615 121.158 90) (layer F.SilkS)
     (effects (font (size 0.6 0.6) (thickness 0.1)))
   )
-  (gr_text R1 (at 187.2615 118.6815 90) (layer F.SilkS)
+  (gr_text R4 (at 187.2615 118.6815 90) (layer F.SilkS)
     (effects (font (size 0.6 0.6) (thickness 0.1)))
   )
