File: AddOns/I2CBoard/I2CBoard.kicad_pcb (KiCad board)
At the start: 2 copper layers, 20 x 30 mm, 17 parts, among them P1 Contacts, P2 Contacts, P6 Contacts, U1 SHT10, U2 TSL2561, U3 BMP180, U4 DHT11, U5 BMP280

Commit message: I²C V1.1 Relay V1.1
Parts:
- added JP3: JUMPER, Connect:GS2, B.Cu at (186.7, 109.7)
- added R3: 10k, Resistors_SMD:R_0805_HandSoldering, F.Cu at (184.3, 119.7)
- U4: value DHT11 -> DHT11/22
Routing:
- net Net-(JP3-Pad1): track 0.00 -> 13.0 mm, vias 0 -> 1
- net /A0: track 0.00 -> 9.14 mm
- net /D6: track 9.76 -> 15.7 mm
- net /VDD: track 57.9 -> 63.1 mm
Other:
- board text added: "HMSensor I²C Board V1.1"
- board text removed: "HMSensor I²C Board V1.0"
