File: AddOns/I2CBoard/I2CBoard.sch (KiCad schematic (older format))
At the start: 15 parts, among them P1 Contacts, P2 Contacts, P6 Contacts, U1 SHT10, U2 TSL2561, U3 BMP180, U4 DHT11, U5 BMP280

Commit message: I²C V1.1 Relay V1.1
Parts:
- added JP3: JUMPER, Connect:GS2, symbol JUMPER
- added R3: 10k, Resistors_SMD:R_0805_HandSoldering, symbol R
Connections:
- net A0: now also JP3.2
- net D6: now also R3.1
- net VDD: now also R3.2
- net at U2.5 (INT): now also JP3.1
Changed lines of the file:
@@
 Title "HMSensor I²C-Board"
 Date ""
-Rev "1.0"
+Rev "1.1"
 Comp ""
-Comment1 "V1.0"
+Comment1 "V1.1"
 Comment2 ""
 Comment3 ""
@@
 	0    1    1    0
 $EndComp
-Wire Wire Line
-	8950 3150 8750 3150
-Wire Wire Line
-	8950 2950 8750 2950
-Wire Wire Line
-	8950 3050 8750 3050
-Wire Wire Line
-	8950 1950 8750 1950
-Wire Wire Line
-	8950 2050 8750 2050
-Wire Wire Line
-	6400 2150 8950 2150
-Wire Wire Line
-	6500 2250 8950 2250
-Wire Wire Line
-	8950 2350 8750 2350
-Wire Wire Line
-	6600 2450 8950 2450
-Wire Wire Line
-	8750 1300 8950 1300
-Wire Wire Line
-	8750 1500 8950 1500
-Wire Wire Line
-	8750 1600 8950 1600
-Wire Wire Line
-	7050 1600 7050 1450
-Connection ~ 7050 1450
-Wire Wire Line
-	7250 1600 7250 1450
-Connection ~ 7250 1450
-Wire Wire Line
-	6750 1450 7850 1450
-Wire Wire Line
-	6500 1650 6500 5050
-Wire Wire Line
-	6500 1650 5900 1650
-Wire Wire Line
-	6500 2600 5900 2600
-Connection ~ 6500 2250
-Wire Wire Line
-	6500 3700 5900 3700
-Connection ~ 6500 2600
-Wire Wire Line
-	6400 1550 5900 1550
-Wire Wire Line
-	6400 2400 5900 2400
-Connection ~ 6400 2150
-Connection ~ 6400 2400
-Wire Wire Line
-	7250 1900 7250 2250
-Connection ~ 7250 2250
-Wire Wire Line
-	7050 1900 7050 2150
-Connection ~ 7050 2150
-Wire Wire Line
-	8950 1400 8500 1400
-Wire Wire Line
-	8500 1400 8500 1200
-Wire Wire Line
-	8500 1200 7950 1200
-Wire Wire Line
-	7950 1700 7950 2850
-Wire Wire Line
-	7950 2850 8950 2850
-Wire Wire Line
-	5900 1750 6100 1750
-Wire Wire Line
-	4800 2400 4400 2400
-Wire Wire Line
-	4400 3700 5100 3700
 $Comp
 L GND #PWR01
@@
 	1    0    0    -1
 $EndComp
-Wire Wire Line
-	5900 1450 6300 1450
-Wire Wire Line
-	6300 1450 6300 1900
-Wire Wire Line
-	4800 2600 4800 3000
-Wire Wire Line
-	3800 2500 4800 2500
-Wire Wire Line
-	4600 2700 4600 2400
-Connection ~ 4600 2400
-Wire Wire Line
-	4600 3000 4600 2900
-Wire Wire Line
-	4600 3700 4600 4000
-Connection ~ 4600 3700
-Wire Wire Line
-	4600 4300 4600 4200
 $Comp
 L GND #PWR05
@@
 	1    0    0    -1
 $EndComp
-Wire Wire Line
-	4800 3300 4800 4300
 Text Label 6750 1450 0    60   ~ 0
 VDD
@@
 Text Label 4400 3700 0    60   ~ 0
 VDD
-Wire Wire Line
-	3550 2600 3300 2600
 $Comp
 L GND #PWR06
@@
 	1    0    0    -1
 $EndComp
-Wire Wire Line
-	4050 2600 4050 3000
 Text Label 3300 2600 0    60   ~ 0
 VDD
@@
 	1    0    0    -1
 $EndComp
-Wire Wire Line
-	6400 3550 5900 3550
-Connection ~ 6400 3550
-Wire Wire Line
-	6400 1550 6400 5250
-Wire Wire Line
-	5100 3850 4600 3850
-Connection ~ 4600 3850
-Wire Wire Line
-	4800 3300 5500 3300
 $Comp
 L DHT11 U4
@@
 	1    0    0    -1
 $EndComp
-Wire Wire Line
-	6600 2450 6600 6400
-Wire Wire Line
-	6600 6400 5750 6400
 $Comp
 L GND #PWR07
@@
 	1    0    0    -1
 $EndComp
-Wire Wire Line
-	5350 6100 5350 5950
-Wire Wire Line
-	5350 6700 5350 6850
 Text Label 5350 5950 3    60   ~ 0
 VDD
@@
 	1    0    0    -1
 $EndComp
-Wire Wire Line
-	6500 5050 6200 5050
-Connection ~ 6500 3700
-Wire Wire Line
-	6400 5250 6200 5250
-Wire Wire Line
-	4700 5250 4700 5650
-Wire Wire Line
-	4700 5250 4800 5250
-Wire Wire Line
-	4800 5450 4700 5450
-Connection ~ 4700 5450
-Wire Wire Line
-	4100 4850 4800 4850
 $Comp
 L C_Small C3
@@
 	1    0    0    -1
 $EndComp
-Wire Wire Line
-	4300 4850 4300 5200
-Connection ~ 4300 4850
-Wire Wire Line
-	4800 5050 4300 5050
-Connection ~ 4300 5050
-Wire Wire Line
-	4300 5650 4300 5400
-Wire Wire Line
-	6200 5450 6300 5450
-Wire Wire Line
-	6300 5450 6300 5650
 Text Label 4100 4850 0    60   ~ 0
 VDD
-Wire Wire Line
-	6200 4850 6200 4700
-Wire Wire Line
-	6200 4700 4700 4700
-Wire Wire Line
-	4700 4700 4700 4850
-Connection ~ 4700 4850
-$Comp
-L GND #PWR?
+$Comp
+L GND #PWR08
 U 1 1 595A2EDD
 P 6300 5650
-F 0 "#PWR?" H 6300 5400 50  0001 C CNN
+F 0 "#PWR08" H 6300 5400 50  0001 C CNN
 F 1 "GND" H 6300 5500 50  0000 C CNN
 F 2 "" H 6300 5650 50  0000 C CNN
@@
 $EndComp
 $Comp
-L GND #PWR?
+L GND #PWR09
 U 1 1 595A2F15
 P 4700 5650
-F 0 "#PWR?" H 4700 5400 50  0001 C CNN
+F 0 "#PWR09" H 4700 5400 50  0001 C CNN
 F 1 "GND" H 4700 5500 50  0000 C CNN
 F 2 "" H 4700 5650 50  0000 C CNN
@@
 $EndComp
 $Comp
-L GND #PWR?
+L GND #PWR010
 U 1 1 595A2F4D
 P 4300 5650
-F 0 "#PWR?" H 4300 5400 50  0001 C CNN
+F 0 "#PWR010" H 4300 5400 50  0001 C CNN
 F 1 "GND" H 4300 5500 50  0000 C CNN
 F 2 "" H 4300 5650 50  0000 C CNN
@@
 	1    0    0    -1
 $EndComp
+$Comp
+L JUMPER JP3
+U 1 1 59A08953
+P 7350 3050
+F 0 "JP3" H 7350 3200 50  0000 C CNN
+F 1 "JUMPER" H 7350 2970 50  0000 C CNN
+F 2 "Connect:GS2" H 7350 3050 50  0001 C CNN
+F 3 "" H 7350 3050 50  0000 C CNN
+	1    7350 3050
+	1    0    0    -1
+$EndComp
+$Comp
+L R R3
+U 1 1 59A6703B
+P 5900 6200
+F 0 "R3" V 5980 6200 50  0000 C CNN
+F 1 "10k" V 5900 6200 50  0000 C CNN
+F 2 "Resistors_SMD:R_0805_HandSoldering" V 5830 6200 50  0001 C CNN
+F 3 "" H 5900 6200 50  0000 C CNN
+	1    5900 6200
+	-1   0    0    1
+$EndComp
+Wire Wire Line
+	8950 3150 8750 3150
+Wire Wire Line
+	8950 2950 8750 2950
+Wire Wire Line
+	8950 3050 8750 3050
+Wire Wire Line
+	8950 1950 8750 1950
+Wire Wire Line
+	8950 2050 8750 2050
+Wire Wire Line
+	6400 2150 8950 2150
+Wire Wire Line
+	6500 2250 8950 2250
+Wire Wire Line
+	8950 2350 8750 2350
+Wire Wire Line
+	6600 2450 8950 2450
+Wire Wire Line
+	8750 1300 8950 1300
+Wire Wire Line
+	8750 1500 8950 1500
+Wire Wire Line
+	8750 1600 8950 1600
+Wire Wire Line
+	7050 1600 7050 1450
+Connection ~ 7050 1450
+Wire Wire Line
+	7250 1600 7250 1450
+Connection ~ 7250 1450
+Wire Wire Line
+	6750 1450 7850 1450
+Wire Wire Line
+	6500 1650 6500 5050
+Wire Wire Line
+	6500 1650 5900 1650
+Wire Wire Line
+	6500 2600 5900 2600
+Connection ~ 6500 2250
+Wire Wire Line
+	6500 3700 5900 3700
+Connection ~ 6500 2600
+Wire Wire Line
+	6400 1550 5900 1550
+Wire Wire Line
+	6400 2400 5900 2400
+Connection ~ 6400 2150
+Connection ~ 6400 2400
+Wire Wire Line
+	7250 1900 7250 2250
+Connection ~ 7250 2250
+Wire Wire Line
+	7050 1900 7050 2150
+Connection ~ 7050 2150
+Wire Wire Line
+	8950 1400 8500 1400
+Wire Wire Line
+	8500 1400 8500 1200
+Wire Wire Line
+	8500 1200 7950 1200
+Wire Wire Line
+	7950 1700 7950 2850
+Wire Wire Line
+	7950 2850 8950 2850
+Wire Wire Line
+	5900 1750 6100 1750
+Wire Wire Line
+	4800 2400 4400 2400
+Wire Wire Line
+	4400 3700 5100 3700
+Wire Wire Line
+	5900 1450 6300 1450
+Wire Wire Line
+	6300 1450 6300 1900
+Wire Wire Line
+	4800 2600 4800 3000
+Wire Wire Line
+	3800 2500 4800 2500
+Wire Wire Line
+	4600 2700 4600 2400
+Connection ~ 4600 2400
+Wire Wire Line
+	4600 3000 4600 2900
+Wire Wire Line
+	4600 3700 4600 4000
+Connection ~ 4600 3700
+Wire Wire Line
+	4600 4300 4600 4200
+Wire Wire Line
+	4800 3300 4800 4300
+Wire Wire Line
+	3550 2600 3300 2600
+Wire Wire Line
+	4050 2600 4050 3000
+Wire Wire Line
+	6400 3550 5900 3550
+Connection ~ 6400 3550
+Wire Wire Line
+	6400 1550 6400 5250
+Wire Wire Line
+	5100 3850 4600 3850
+Connection ~ 4600 3850
+Wire Wire Line
+	4800 3300 5500 3300
+Wire Wire Line
+	6600 2450 6600 6400
+Wire Wire Line
+	6600 6400 5750 6400
+Wire Wire Line
+	5350 6100 5350 5950
+Wire Wire Line
+	5350 6700 5350 6850
+Wire Wire Line
+	6500 5050 6200 5050
+Connection ~ 6500 3700
+Wire Wire Line
+	6400 5250 6200 5250
+Wire Wire Line
+	4700 5250 4700 5650
+Wire Wire Line
+	4700 5250 4800 5250
+Wire Wire Line
+	4800 5450 4700 5450
+Connection ~ 4700 5450
+Wire Wire Line
+	4100 4850 4800 4850
+Wire Wire Line
+	4300 4850 4300 5200
+Connection ~ 4300 4850
+Wire Wire Line
+	4800 5050 4300 5050
+Connection ~ 4300 5050
+Wire Wire Line
+	4300 5650 4300 5400
+Wire Wire Line
+	6200 5450 6300 5450
+Wire Wire Line
+	6300 5450 6300 5650
+Wire Wire Line
+	6200 4850 6200 4700
+Wire Wire Line
+	6200 4700 4700 4700
+Wire Wire Line
+	4700 4700 4700 4850
+Connection ~ 4700 4850
+Wire Wire Line
+	7650 3050 8800 3050
+Connection ~ 8800 3050
+Wire Wire Line
+	7050 3050 7050 2500
+Wire Wire Line
+	7050 2500 5900 2500
+Wire Wire Line
+	5900 6350 5900 6400
+Connection ~ 5900 6400
+Wire Wire Line
+	5900 6050 5900 6000
+Wire Wire Line
+	5900 6000 5350 6000
+Connection ~ 5350 6000
 $EndSCHEMATC
